Commit message: Implemented computeSekeleton function in RobotCollisionState. Added useful getters for this purpose: getLinLeafSpheresIndices, getSpheresStates, and getGroupStates. Optimized distance query function - getCollisionDistance in SelfCollisionModel.

File: smpl_test/2DoF_planar/planar_2dof_mini.urdf (robot description, URDF)
Before this commit: robot planar_2dof_mini, 4 links, 3 joints
Joints:
- joint joint2: origin xyz=0.25 0 0 rpy=0 0 0 -> xyz=0.20 0 0 rpy=0 0 0

Commit message: Bur implementation works. Needs a lot of optimization.

File: smpl_test/2DoF_planar/planar_2dof_mini.urdf (robot description, URDF)
Before this commit: robot planar_2dof_mini, 4 links, 3 joints
Links:
- link link1: geometry collision sphere radius=0.05; collision sphere radius=0.05
- link link2: geometry collision sphere radius=0.05; collision sphere radius=0.05
