Commit message: Fixed planar_2DoF urdf and configs.

File: smpl_test/planar_arm/planar_2dof.urdf (robot description, URDF)
Before this commit: robot planar_2dof, 4 links, 3 joints
Links:
- link base_link: geometry collision sphere radius=0.1; visual cylinder length=0.2 radius=0.1
- link link1: geometry collision sphere radius=0.05; collision sphere radius=0.05
- link link2: geometry collision sphere radius=0.05; collision sphere radius=0.05
Joints:
- joint joint2: origin xyz=0.45 0 0 rpy=0 0 0 -> xyz=0.20 0 0 rpy=0 0 0
